File: project/ZSWatch-HeartRate.kicad_sch (KiCad schematic)
At the start: 17 parts, among them IC101 MAX32664, IC102 MAXM86161, X101 Mainboard, Y101 32kHz

Commit message: Fix CI/CD errors
Parts:
- C101, C102, C103, C104, C105, C106, C107, IC101, IC102, R101, R102, R103, R104, R105, R106, X101, Y101: CONFIG (none) -> Full
Changed lines of the file:
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@@
       (effects (font (size 1.27 1.27)) hide)
     )
-    (property "CONFIG" "" (at 118.11 73.66 0)
+    (property "CONFIG" "Full" (at 118.11 73.66 0)
       (effects (font (size 1.27 1.27)) hide)
     )
@@
       (effects (font (size 1.27 1.27)) hide)
     )
-    (property "CONFIG" "" (at 36.83 116.84 0)
+    (property "CONFIG" "Full" (at 36.83 116.84 0)
       (effects (font (size 1.27 1.27)) hide)
     )
@@
       (effects (font (size 1.27 1.27)) hide)
     )
-    (property "CONFIG" "" (at 105.41 113.03 0)
+    (property "CONFIG" "Full" (at 105.41 113.03 0)
       (effects (font (size 1.27 1.27)) hide)
     )
@@
       (effects (font (size 1.27 1.27)) hide)
     )
-    (property "CONFIG" "" (at 147.32 97.79 0)
+    (property "CONFIG" "Full" (at 147.32 97.79 0)
       (effects (font (size 1.27 1.27)) hide)
     )
@@
       (effects (font (size 1.27 1.27)) hide)
     )
-    (property "CONFIG" "" (at 226.06 90.17 0)
+    (property "CONFIG" "Full" (at 226.06 90.17 0)
       (effects (font (size 1.27 1.27)) hide)
     )
@@
       (effects (font (size 1.27 1.27)) hide)
     )
-    (property "CONFIG" "" (at 105.41 104.14 0)
+    (property "CONFIG" "Full" (at 105.41 104.14 0)
       (effects (font (size 1.27 1.27)) hide)
     )
@@
       (effects (font (size 1.27 1.27)) hide)
     )
-    (property "CONFIG" "" (at 123.19 110.49 0)
+    (property "CONFIG" "Full" (at 123.19 110.49 0)
       (effects (font (size 1.27 1.27)) hide)
     )
@@
       (effects (font (size 1.27 1.27)) hide)
     )
-    (property "CONFIG" "" (at 176.53 81.28 0)
+    (property "CONFIG" "Full" (at 176.53 81.28 0)
       (effects (font (size 1.27 1.27)) hide)
     )
@@
       (effects (font (size 1.27 1.27)) hide)
     )
-    (property "CONFIG" "" (at 173.99 81.28 0)
+    (property "CONFIG" "Full" (at 173.99 81.28 0)
       (effects (font (size 1.27 1.27)) hide)
     )
@@
       (effects (font (size 1.27 1.27)) hide)
     )
-    (property "CONFIG" "" (at 194.31 73.66 0)
+    (property "CONFIG" "Full" (at 194.31 73.66 0)
       (effects (font (size 1.27 1.27)) hide)
     )
@@
       (effects (font (size 1.27 1.27)) hide)
     )
-    (property "CONFIG" "" (at 138.43 68.58 0)
+    (property "CONFIG" "Full" (at 138.43 68.58 0)
       (effects (font (size 1.27 1.27)) hide)
     )
@@
       (effects (font (size 1.27 1.27)) hide)
     )
-    (property "CONFIG" "" (at 205.74 58.42 0)
+    (property "CONFIG" "Full" (at 205.74 58.42 0)
       (effects (font (size 1.27 1.27)) hide)
     )
@@
       (effects (font (size 1.27 1.27)) hide)
     )
-    (property "CONFIG" "" (at 153.67 69.85 0)
+    (property "CONFIG" "Full" (at 153.67 69.85 0)
       (effects (font (size 1.27 1.27)) hide)
     )
@@
       (effects (font (size 1.27 1.27)) hide)
     )
-    (property "CONFIG" "" (at 143.51 43.18 0)
+    (property "CONFIG" "Full" (at 143.51 43.18 0)
       (effects (font (size 1.27 1.27)) hide)
     )
@@
       (effects (font (size 1.27 1.27)) hide)
     )
-    (property "CONFIG" "" (at 120.65 73.66 0)
+    (property "CONFIG" "Full" (at 120.65 73.66 0)
       (effects (font (size 1.27 1.27)) hide)
     )
@@
       (effects (font (size 1.27 1.27)) hide)
     )
-    (property "CONFIG" "" (at 200.66 100.33 0)
+    (property "CONFIG" "Full" (at 200.66 100.33 0)
       (effects (font (size 1.27 1.27)) hide)
     )
@@
       (effects (font (size 1.27 1.27)) hide)
     )
-    (property "CONFIG" "" (at 207.01 77.47 0)
-      (effects (font (size 1.27 1.27)) hide)
-    )
+    (property "CONFIG" "Full" (at 207.01 77.47 0)
+      (effects (font (size 1.27 1.27)) hide)
+    )

Commit message: - Working on version 1
Parts:
- IC102: footprint AnalogDevices:MAXM86161 -> AnalogDevices:MAXM8616
- X101: Distributor Digikey -> Mouser; Order Number 609-101R014FB110CT-ND -> 649-101R014FB110
Connections:
- net INT_ACC: now also X101.3 (Pin_3); no longer X101.1 (Pin_1)
- net INT_HR: now also X101.1 (Pin_1)
- net SDA: now also X101.7 (Pin_7); no longer X101.9 (Pin_9)
- net MFIO: now reaches IC101.1 (MFIO)
- net MFIO: now also X101.9 (Pin_9)
- net V_Bat renamed V_LED
- no-connect marks 1 -> 5
Other:
- moved on the sheet: R106

Commit message: First dev board version
Parts:
- removed C103, C104, C105, C106, C107: 1u, Capacitor_SMD:C_0603_1608Metric_Pad1.08x0.95mm_HandSolder, symbol Device:C
- removed IC101: MAX32664, Package_DFN_QFN:QFN-24-1EP_3x3mm_P0.4mm_EP1.75x1.6mm, symbol AnalogDevices_Kampi:MAX32664
- removed IC102: MAXM86161, AnalogDevices:MAXM8616, symbol AnalogDevices_Kampi:MAXM86161
- removed R101: 10R, Resistor_SMD:R_0603_1608Metric_Pad0.98x0.95mm_HandSolder, symbol Device:R
- removed R102, R104: 4k7, Resistor_SMD:R_0603_1608Metric_Pad0.98x0.95mm_HandSolder, symbol Device:R
- removed X101: Mainboard, Amphenol:101R014FB110, symbol Connector_Generic_Shielded:Conn_01x14_Shielded
- added C103, C114, C116: 100n, Capacitor_SMD:C_0402_1005Metric, symbol Device:C_Small
- added C104, C111, C112: 1u, Capacitor_SMD:C_0402_1005Metric, symbol Device:C_Small
- added C105: 22u, Capacitor_SMD:C_0402_1005Metric, symbol Device:C_Small
- added C106, C115: 10u, Capacitor_SMD:C_0402_1005Metric, symbol Device:C_Small
- added C107: 2u2, Capacitor_SMD:C_0603_1608Metric, symbol Device:C_Small
- added C108: 4u7, Capacitor_SMD:C_0603_1608Metric, symbol Device:C_Small
- added C109: 100n, Capacitor_SMD:C_0603_1608Metric, symbol Device:C_Small
- added C110, C113: 1u, Capacitor_SMD:C_0603_1608Metric, symbol Device:C
- added D102: D_Photo, Vishay:VEMD5080X01, symbol Device:D_Photo
- added D104: RED, Diode_SMD:D_0603_1608Metric, symbol Device:LED
- added D105: IR, Diode_SMD:D_0603_1608Metric, symbol Device:LED
- added D106: GREEN, Diode_SMD:D_0603_1608Metric, symbol Device:LED
- added D107: STATUS, LED_SMD:LED_0805_2012Metric_Pad1.15x1.40mm_HandSolder, symbol Device:LED
- added IC101: LIS2DS12, Package_LGA:LGA-12_2x2mm_P0.5mm, symbol ST:LIS2DS12
- added IC102: MCP73832-2-OT, Package_TO_SOT_SMD:SOT-23-5, symbol Battery_Management:MCP73832-2-OT
- added IC103: MAX32664, Package_BGA_Kampi:WLP-16_2x2mm_P0.5mm, symbol Analog Devices:MAX32664-SPI-WLP
- added IC104: TPS61240, Package_BGA_Kampi:DSBGA-6_0.886x1.288mm_2x3_P0.4mm, symbol Texas Instruments:TPS61240-BGA
- added IC105: MAX86141, Package_BGA_Kampi:THIN-WLP-20_2.228x1.967mm_P0.4mm, symbol Analog Devices:MAX86141
- added IC106: MIC5365-1.8, Package_TO_SOT_SMD:SOT-23-5, symbol Microchip_Kampi:MIC5365
- added J101: SPI, Connector_PinHeader_2.54mm:PinHeader_1x06_P2.54mm_Vertical, symbol Connector_Generic:Conn_01x06
- added J102: GPIO, Connector_PinHeader_2.54mm:PinHeader_1x07_P2.54mm_Vertical, symbol Connector_Generic:Conn_01x07
- added J103: UART, Connector_PinHeader_2.54mm:PinHeader_1x03_P2.54mm_Vertical, symbol Connector_Generic:Conn_01x03
- added J104: I2C, Connector_PinHeader_2.54mm:PinHeader_1x03_P2.54mm_Vertical, symbol Connector_Generic:Conn_01x03
- added L101: 1u, Inductor_SMD:L_0603_1608Metric, symbol Device:L
- added M101: BM15C, Fanstel:BM15C, symbol Fanstel:BM15C
- added R101, R108: 10k, Capacitor_SMD:C_0603_1608Metric, symbol Device:R_Small
- added R102, R104: 5k1, Resistor_SMD:R_0603_1608Metric, symbol Device:R_Small
- added R107: 10k, Capacitor_SMD:C_0603_1608Metric, symbol Device:R
- added R109: 0R, Resistor_SMD:R_0805_2012Metric, symbol Device:R
- added SW101: BTN1, Wuerth:WS-TASV-6x6, symbol Switch:SW_MEC_5E
- added SW102: RESET, Wuerth:WS-TASV-6x6, symbol Switch:SW_MEC_5E
- added X102: CHARGE, Connector_USB:USB_C_Receptacle_GCT_USB4105-xx-A_16P_TopMnt_Horizontal, symbol Connector:USB_C_Receptacle_USB2.0_14P
- added X103: BATTERY, Molex:78171-0002, symbol Connector_Generic:Conn_01x02
- added X104: DEBUG, Connector_PinHeader_1.27mm:PinHeader_2x05_P1.27mm_Vertical, symbol Connector:Conn_ARM_JTAG_SWD_10
- C101: value 100n -> 4u7; footprint Capacitor_SMD:C_0603_1608Metric_Pad1.08x0.95mm_HandSolder -> Capacitor_SMD:C_0603_1608Metric; CONFIG Full -> (none); Distributor Mouser -> (none); Mfr. KEMET -> (none); Mfr. No. C0603C104K8RAC -> (none); Order Number 80-C0603C104K8RAC -> (none)
- C102: value 1u -> 4u7; footprint Capacitor_SMD:C_0603_1608Metric_Pad1.08x0.95mm_HandSolder -> Capacitor_SMD:C_0603_1608Metric; CONFIG Full -> (none); Distributor Mouser -> (none); Mfr. KEMET -> (none); Mfr. No. C0603C105K8RAC -> (none); Order Number 80-C0603C105K8RAC -> (none)
- R103: footprint Resistor_SMD:R_0603_1608Metric_Pad0.98x0.95mm_HandSolder -> Resistor_SMD:R_0402_1005Metric; CONFIG Full -> (none); Distributor Mouser -> (none); Mfr. Bourns -> (none); Mfr. No. CR0603-JW-472ELF -> (none); Order Number 652-CR0603-JW-472ELF -> (none); now fitted
- R105: value 4k7 -> 220R; footprint Resistor_SMD:R_0603_1608Metric_Pad0.98x0.95mm_HandSolder -> Capacitor_SMD:C_0603_1608Metric; CONFIG Full -> (none); Distributor Mouser -> (none); Mfr. Bourns -> (none); Mfr. No. CR0603-JW-472ELF -> (none); Order Number 652-CR0603-JW-472ELF -> (none); manf (none) -> Bourns; manf# (none) -> CR0402-JW-221GLF; mouser# (none) -> 652-CR0402-JW-221GLF
- R106: value 4k7 -> 10k; footprint Resistor_SMD:R_0603_1608Metric_Pad0.98x0.95mm_HandSolder -> Capacitor_SMD:C_0603_1608Metric; CONFIG Full -> (none); Distributor Mouser -> (none); Mfr. Bourns -> (none); Mfr. No. CR0603-JW-472ELF -> (none); Order Number 652-CR0603-JW-472ELF -> (none)
- Y101: footprint Crystal:Crystal_SMD_3215-2Pin_3.2x1.5mm -> Crystal_Kampi:ECS_ECX-1210; CONFIG Full -> (none); Distributor Mouser -> (none); Mfr. ABRACON -> (none); Mfr. No. ABS07-32.768KHZ-6-T -> (none); Order Number 815-ABS07-32.768K6T -> (none)
Connections:
- net INT_HR is gone; now on net GND: R106.2
- net +1V8: now also C103.1, C105.1, C109.1, C110.1, C111.1, C114.1, C115.1, C116.1, IC101.10 (VDD_{IO}), IC101.9 (VDD), IC103.A3 (V_{DD}), IC105.C2 (DVDD), IC105.D2 (AVDD), IC106.5 (OUT), J102.7 (Pin_7), M101.B8 (VDD), M101.C8 (VDD), R107.2, R108.1, X104.1 (VTref); no longer C102.1, R105.1, R106.1
- net GND: now also C101.2, C103.2, C104.2, C105.2, C106.2, C107.2, C108.2, C109.2, C110.2, C111.2, C112.2, C113.2, C114.2, C115.2, C116.2, D102.2 (A), IC101.6 (GND), IC101.7 (RES), IC101.8 (GND), IC102.2 (V_{SS}), IC103.B2 (GND), IC104.A2 (GND), IC105.C3 (DGND), IC105.C4 (AGND), IC105.C5 (PD_GND), IC105.D3 (PGND), IC105.D4 (PD2_IN), IC106.2 (GND), J101.1 (Pin_1), J102.1 (Pin_1), J103.3 (Pin_3), J104.3 (Pin_3), M101.A1 (GND), M101.A9 (GND), M101.B1 (GND), M101.B7 (GND), M101.B9 (GND), M101.D1 (GND), M101.E1 (GND), M101.F1 (GND), M101.H8 (GND), R101.2, R102.2, R104.1, SW101.1, SW101.2, SW102.3 (K), SW102.4 (A), X102.A1 (GND), X102.A12 (GND), X102.B1 (GND), X102.B12 (GND), X102.S1 (SHIELD), X103.2 (Pin_2), X104.3 (GND), X104.5 (GND)
- net SCL: now also IC103.D1 (SCL), J104.2 (Pin_2), M101.K6 (P2.08)
- net SDA: now also IC103.D2 (SDA), J104.1 (Pin_1), M101.K5 (P2.10); no longer R103.2
- net ~{RESET}: now also M101.G2 (~{RESET}), R108.2, SW102.1, SW102.2, X104.10 (~{RESET}); no longer C101.1
- net at R105.2: now also D107.2 (A)
- net at Y101.2: now also IC103.A2 (32k_{IN})
- net at Y101.1: now also IC103.A1 (32k_{OUT})
- new net: M101.K7 (P2.06), R109.1
- new net: D106.1 (K), IC105.B1 (LED3_DRV)
- new net: C112.1, IC103.A4 (V_{CORE})
- new net: M101.J7 (P2.03), SW101.3 (K), SW101.4 (A)
- new net: C101.1, IC102.4 (V_{DD}), X102.A4 (VBUS), X102.A9 (VBUS), X102.B4 (VBUS), X102.B9 (VBUS)
- new net: IC102.5 (PROG), R106.1
- new net: IC101.1 (SCL/SCLK), IC103.C3 (SCLK_{SENSOR}), IC105.A2 (SCLK), J101.2 (Pin_2)
- new net: IC101.4 (SDA/SDI/SDO), IC103.D4 (MOSI_{SENSOR}), IC105.A4 (MOSI), J101.3 (Pin_3)
- new net: IC101.3 (SDO/ADDR0), IC103.D3 (MISO_{SENSOR}), IC105.A3 (MISO), J101.4 (Pin_4)
- new net: IC101.2 (CS), IC103.C1 (CS_{ACC}), J101.5 (Pin_5)
- new net: IC103.C4 (CS_{PPG}), IC105.A5 (~{CSB}), J101.6 (Pin_6)
- new net: IC103.B4 (INT_{PPG}), IC105.B2 (~{INT}), R103.2
- new net: C104.1, IC105.B5 (VREF)
- new net: D104.1 (K), IC105.C1 (LED2_DRV)
- new net: D105.1 (K), IC105.D1 (LED1_DRV)
- new net: D102.1 (K), IC105.D5 (PD1_IN)
- new net: R102.1, X102.A5 (CC1)
- new net: R104.2, X102.B5 (CC2)
- new net: J102.2 (Pin_2), M101.H2 (P0.04)
- new net: J102.3 (Pin_3), M101.K4 (P0.01)
- new net: J102.4 (Pin_4), M101.K2 (P0.02)
- new net: J102.5 (Pin_5), M101.J4 (P0.00)
- new net: J102.6 (Pin_6), M101.J2 (P0.03)
- new net: IC104.B1 (L), L101.2
- new net: D107.1 (K), M101.K8 (P2.05)
- new net: J103.1 (Pin_1), M101.F8 (P1.05/AIN1)
- new net +BATT: R105.1
- new net CHARGE: IC102.1 (STAT), M101.J6 (P2.07), R107.1
- new net ENABLE_{LED}: IC104.C1 (EN), R109.2
- new net INT_{ACC}: IC101.12 (INT1), IC103.B3 (INT_{ACC})
- new net STATUS: IC103.C2 (MFIO), M101.J9 (P2.01)
- new net SWDCLK: M101.K3 (SWDCLK), X104.4 (SWDCLK/TCK)
- new net SWDIO: M101.J3 (SWDIO), X104.2 (SWDIO/TMS)
- new net TxD: J103.2 (Pin_2), M101.E8 (P1.03/NFC)
- new net V_{BAT}: C102.1, C107.1, C113.1, IC102.3 (V_{BAT}), IC104.A1 (IN), IC106.1 (IN), IC106.3 (EN), L101.1, X103.1 (Pin_1)
- new net V_{LED}: C106.1, C108.1, D104.2 (A), D105.2 (A), D106.2 (A), IC104.B2 (OUT), IC104.C2 (FB), IC105.A1 (V_{LED})
- new net ~{RESET_{HR}}: IC103.B1 (~{RESET}), M101.H9 (P2.00), R101.1
- no-connect marks 5 -> 26
Other:
- note added: "557 nm"
- note added: "660 nm"
- note added: "880 nm"
- note added: "Layout guidelines for MAX8614x: - Connect all GNDs to a single ground plane and use one single via to PCB ground - Use different vias for all decoupling caps - PD_IN must be shielded by PD_GND - PD_GND on the layer where the MAX8614x is mounted, PG_IN under PD_GND - No traces over or under PD_GND"
- note added: "TODO: Can we use GPIO1 or 2 to Enable / Disable VLED?"
- company: github.com/jakkra/ZSWatch-HeartRate -> github.com/...
- title: ZSWatch Heart rate -> ZSWatch Heart Rate Dev-Board

Commit message: Update CI/CD pipeline
Parts:
- added C117: 1u, Capacitor_SMD:C_0402_1005Metric, symbol Device:C_Small
- C101, C102, C108: manf (none) -> TAIYO YUDEN; manf# (none) -> LMK107BJ475KA-T; mouser# (none) -> 963-LMK107BJ475KA-T
- C103, C114, C116: manf (none) -> KEMET; manf# (none) -> C0402C104K4RAC7411; mouser# (none) -> 80-C0402C104K4R7411
- C105: manf (none) -> TAIYO YUDEN; manf# (none) -> MEASP105CC6226MF1A01; mouser# (none) -> 963-MEASP105CC62261A
- C106, C115: manf (none) -> TAIYO YUDEN; manf# (none) -> AMK105CBJ106MV-F; mouser# (none) -> 963-AMK105CBJ106MV-F
- C107: manf (none) -> KYOCERA AVX; manf# (none) -> 06033D225MAT2A; mouser# (none) -> 581-06033D225MAT2A
- C109: footprint Capacitor_SMD:C_0603_1608Metric -> Capacitor_SMD:C_0402_1005Metric; manf (none) -> KEMET; manf# (none) -> C0402C104K4RAC7411; mouser# (none) -> 80-C0402C104K4R7411
- D104: value RED -> IR; manf VCC -> Kingbright; manf# 7017X1 -> APTD1608SF4C; mouser# 606-7017X1 -> 604-APTD1608SF4C
- D105: value IR -> GREEN; manf Kingbright -> Bivar; manf# APTD1608SF4C -> SM0603PGC; mouser# 604-APTD1608SF4C -> 749-SM0603PGC
- D106: value GREEN -> RED; manf Bivar -> VCC; manf# SM0603PGC -> 7017X1; mouser# 749-SM0603PGC -> 606-7017X1
- IC103: footprint Package_BGA_Kampi:WLP-16_2x2mm_P0.5mm -> Package_DFN_QFN:QFN-24-1EP_3x3mm_P0.4mm_EP1.75x1.6mm; symbol Analog Devices:MAX32664-SPI-WLP -> Analog Devices:MAX32664-SPI-TQFN
- IC106: manf# MIC5365-1.8YC5-TR -> MIC5365-1.8YD5-TR; mouser# 998-MIC5365-1.8YC5-TR -> 998- MIC5365-1.8YD5-TR
- J104: footprint Connector_PinHeader_2.54mm:PinHeader_1x03_P2.54mm_Vertical -> Connector_PinHeader_2.54mm:PinHeader_1x04_P2.54mm_Vertical; symbol Connector_Generic:Conn_01x03 -> Connector_Generic:Conn_01x04
- R101, R106, R107, R108: footprint Capacitor_SMD:C_0603_1608Metric -> Resistor_SMD:R_0402_1005Metric; manf (none) -> Bourns; manf# (none) -> CR0402-JW-103GLF; mouser# (none) -> 652-CR0402-JW-103GLF
- R102, R104: footprint Resistor_SMD:R_0603_1608Metric -> Resistor_SMD:R_0402_1005Metric; manf (none) -> Bourns; manf# (none) -> CR0402-FX-5101GLF; mouser# (none) -> 652-CR0402-FX-5101GLF
- R103: manf (none) -> YAGEO; manf# (none) -> RC0402FR-7D4K7L; mouser# (none) -> 603-RC0402FR-7D4K7L
- SW101, SW102: symbol Switch:SW_MEC_5E -> Switch:SW_DPST
- X103: manf (none) -> Molex; manf# (none) -> 78171-0002; mouser# (none) -> 538-78171-0002
- Y101: manf (none) -> ECS; manf# (none) -> ECS-.327-6-1210-TR; mouser# (none) -> 520-.327-6-1210-TR
Connections:
- net +1V8: now also IC103.11 (V_{DD}), IC103.22 (V_{DD}), C117.1; no longer IC103.A3 (V_{DD})
- net GND: now also IC103.10 (GND), IC103.7 (GND), J104.4 (Pin_4), SW101.3, SW102.2, C117.2; no longer IC103.B2 (GND), J104.3 (Pin_3), SW101.2, SW102.3 (K)
- net INT_{ACC}: now also IC103.13 (INT_{ACC}); no longer IC103.B3 (INT_{ACC})
- net SCL: now also IC103.24 (SCL); no longer IC103.D1 (SCL)
- net SDA: now also IC103.23 (SDA); no longer IC103.D2 (SDA)
- net STATUS: now also IC103.1 (MFIO); no longer IC103.C2 (MFIO)
- net ~{RESET_{HR}}: now also IC103.6 (~{RESET}), J104.3 (Pin_3); no longer IC103.B1 (~{RESET})
- net ~{RESET}: now also SW102.3; no longer SW102.2
- net at C112.1: now also IC103.12 (V_{CORE}); no longer IC103.A4 (V_{CORE})
- net at M101.J7 (P2.03), SW101.4: now also SW101.2; no longer SW101.3 (K)
- net at Y101.1: now also IC103.8 (32k_{OUT}); no longer IC103.A1 (32k_{OUT})
- net at Y101.2: now also IC103.9 (32k_{IN}); no longer IC103.A2 (32k_{IN})
- net at IC101.1 (SCL/SCLK), IC105.A2 (SCLK): now also IC103.19 (SCLK_{SENSOR}), J101.4 (Pin_4); no longer IC103.C3 (SCLK_{SENSOR}), J101.2 (Pin_2)
- net at IC101.4 (SDA/SDI/SDO), IC105.A4 (MOSI): now also IC103.20 (MOSI_{SENSOR}), J101.2 (Pin_2); no longer IC103.D4 (MOSI_{SENSOR}), J101.3 (Pin_3)
- net at IC101.3 (SDO/ADDR0), IC105.A3 (MISO): now also IC103.21 (MISO_{SENSOR}), J101.3 (Pin_3); no longer IC103.D3 (MISO_{SENSOR}), J101.4 (Pin_4)
- net at IC101.2 (CS), J101.5 (Pin_5): now also IC103.2 (CS_{ACC}); no longer IC103.C1 (CS_{ACC})
- net at IC105.A5 (~{CSB}), J101.6 (Pin_6): now also IC103.18 (CS_{PPG}); no longer IC103.C4 (CS_{PPG})
- net at IC105.B2 (~{INT}), R103.2: now also IC103.14 (INT_{PPG}); no longer IC103.B4 (INT_{PPG})

Commit message: Fix wrong MAX32664 footprint
Parts:
- IC103: footprint Package_DFN_QFN:QFN-24-1EP_3x3mm_P0.4mm_EP1.75x1.6mm -> Analog Devices:MAX32664GTG; manf (none) -> Analog Devices / Maxim Integrated; manf# MAX32664GWEC+ -> MAX32664GTGC+; mouser# (none) -> 700-MAX32664GTGC+
Changed lines of the file:
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@@
 			)
 		)
-		(property "Footprint" "Package_DFN_QFN:QFN-24-1EP_3x3mm_P0.4mm_EP1.75x1.6mm"
+		(property "Footprint" "Analog Devices:MAX32664GTG"
 			(at 193.04 135.89 0)
 			(effects
@@
 			)
 		)
-		(property "Datasheet" "https://www.analog.com/media/en/technical-documentation/data-sheets/MAX32664.pdf"
+		(property "Datasheet" "https://www.mouser.de/datasheet/2/609/MAX32664-3469756.pdf"
 			(at 193.04 135.89 0)
 			(effects
@@
 			)
 		)
-		(property "manf" ""
+		(property "manf" "Analog Devices / Maxim Integrated"
 			(at 193.04 135.89 0)
 			(effects
@@
 			)
 		)
-		(property "manf#" "MAX32664GWEC+ "
+		(property "manf#" "MAX32664GTGC+"
 			(at 193.04 135.89 0)
 			(effects
@@
 			)
 		)
-		(property "mouser#" ""
+		(property "mouser#" "700-MAX32664GTGC+"
 			(at 193.04 135.89 0)
 			(effects
