File: devkit/ZSWatch-Heartrate-DevKit.kicad_pcb (KiCad board)
At the start: 4 copper layers, 45 x 36.9 mm, 49 parts, among them IC401 MIC5365-1.8, IC402 TPS61240, IC403 MCP73832-2-OT, IC404 MAX32664, IC405 MAX86141, IC406 LIS2DS12, J401 I2C, J402 SPI, M401 BM15C, Q401 BSS138, SW401 RESET, SW402 BTN1, X401 CHARGE, X402 BATTERY, X403 DEBUG, Y401 32kHz

Commit message: Update outputs (release)
Other:
- board text added: "0.196mm"
- board text added: "0.43mm"
- board text added: "Inner1"
- board text added: "Inner2"
- board text added: "Plane"
- board text added: "Prepreg"
- board text added: "Total thickness: 0.982mm"
- board text removed: "1.51mm"
- board text removed: "Total thickness: 1.6mm"
