File: devkit/Main.kicad_sch (KiCad schematic)
At the start: 49 parts, among them IC401 MIC5365-1.8, IC402 TPS61240, IC403 MCP73832-2-OT, IC404 MAX32664, IC405 MAX86141, IC406 LIS2DS12, J401 I2C, J402 SPI, M401 BM15C, Q401 BSS138, SW401 RESET, SW402 BTN1, X401 CHARGE, X402 BATTERY, X403 DEBUG, Y401 32kHz

Commit message: Bug: Issue #17
- Wrong part number for SWD connector

Closes: #17

Signed-off-by: Daniel Kampert <DanielKampert@kampis-elektroecke.de>
Parts:
- X403: manf# 623310235521 -> 62201021121; mouser# 710-623310235521 -> 710-62201021121
Changed lines of the file:
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@@
 			)
 		)
-		(property "manf#" "623310235521"
+		(property "manf#" "62201021121"
 			(at 191.77 260.35 0)
 			(effects
@@
 			)
 		)
-		(property "mouser#" "710-623310235521"
+		(property "mouser#" "710-62201021121"
 			(at 191.77 260.35 0)
 			(effects
